File: Schematica/AutoMicrophone.kicad_sch (KiCad schematic)
At the start: 22 parts, among them J1 XLR3_Input, J2 XLR3_Output, J3 Jack-DC, Q1 IRLZ44N, Q2 IRLZ44N, Q3 2N3904, U1 SPX2920U-5.0_TO220, U2 LM358, U3 ATtiny85-20P

Commit message: Rev 4
Parts:
- added R9: 100, symbol Device:R
Connections:
- net CONTROL: now also R9.1; no longer Q1.1 (G), Q2.1 (G), R3.2
- new net: Q1.1 (G), Q2.1 (G), R3.2, R9.2
Other:
- moved on the sheet: R3
Changed lines of the file:
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@@
     (title "AutoMicrophone")
     (date "2022-09-24")
-    (rev "2")
+    (rev "4")
     (company "Aeindus")
   )
@@
   (junction (at 60.96 62.23) (diameter 0) (color 0 0 0 0)
   )
-  (junction (at 80.01 27.94) (diameter 0) (color 0 0 0 0)
-  )
-  (junction (at 80.01 52.07) (diameter 0) (color 0 0 0 0)
-  )
   (junction (at 25.4 107.95) (diameter 0) (color 0 0 0 0)
   )
@@
   (junction (at 200.66 90.17) (diameter 0) (color 0 0 0 0)
   )
+  (junction (at 82.55 27.94) (diameter 0) (color 0 0 0 0)
+  )
   (junction (at 100.33 41.91) (diameter 0) (color 0 0 0 0)
   )
@@
   (junction (at 58.42 107.95) (diameter 0) (color 0 0 0 0)
   )
+  (junction (at 82.55 52.07) (diameter 0) (color 0 0 0 0)
+  )
   (wire (pts (xy 116.84 96.52) (xy 116.84 91.44))
     (stroke (width 0) (type default) (color 0 0 0 0))
   )
+  (wire (pts (xy 44.45 27.94) (xy 82.55 27.94))
+    (stroke (width 0) (type default) (color 0 0 0 0))
+  )
   (wire (pts (xy 240.03 118.11) (xy 240.03 123.19))
     (stroke (width 0) (type default) (color 0 0 0 0))
   )
-  (wire (pts (xy 71.12 52.07) (xy 80.01 52.07))
-    (stroke (width 0) (type default) (color 0 0 0 0))
-  )
   (wire (pts (xy 143.51 88.9) (xy 149.86 88.9))
     (stroke (width 0) (type default) (color 0 0 0 0))
@@
     (stroke (width 0) (type default) (color 0 0 0 0))
   )
+  (wire (pts (xy 82.55 52.07) (xy 92.71 52.07))
+    (stroke (width 0) (type default) (color 0 0 0 0))
+  )
   (wire (pts (xy 250.19 97.79) (xy 250.19 90.17))
     (stroke (width 0) (type default) (color 0 0 0 0))
@@
     (stroke (width 0) (type default) (color 0 0 0 0))
   )
-  (wire (pts (xy 80.01 52.07) (xy 92.71 52.07))
+  (wire (pts (xy 78.74 52.07) (xy 82.55 52.07))
     (stroke (width 0) (type default) (color 0 0 0 0))
   )
@@
     (stroke (width 0) (type default) (color 0 0 0 0))
   )
+  (wire (pts (xy 82.55 27.94) (xy 90.17 27.94))
+    (stroke (width 0) (type default) (color 0 0 0 0))
+  )
   (wire (pts (xy 58.42 107.95) (xy 74.93 107.95))
     (stroke (width 0) (type default) (color 0 0 0 0))
@@
     (stroke (width 0) (type default) (color 0 0 0 0))
   )
+  (wire (pts (xy 67.31 52.07) (xy 71.12 52.07))
+    (stroke (width 0) (type default) (color 0 0 0 0))
+  )
   (wire (pts (xy 123.19 49.53) (xy 123.19 62.23))
     (stroke (width 0) (type default) (color 0 0 0 0))
   )
-  (wire (pts (xy 44.45 27.94) (xy 80.01 27.94))
-    (stroke (width 0) (type default) (color 0 0 0 0))
-  )
   (wire (pts (xy 191.77 46.99) (xy 199.39 46.99))
     (stroke (width 0) (type default) (color 0 0 0 0))
@@
     (stroke (width 0) (type default) (color 0 0 0 0))
   )
-  (wire (pts (xy 80.01 27.94) (xy 90.17 27.94))
-    (stroke (width 0) (type default) (color 0 0 0 0))
-  )
   (wire (pts (xy 107.95 91.44) (xy 116.84 91.44))
     (stroke (width 0) (type default) (color 0 0 0 0))
@@
     (stroke (width 0) (type default) (color 0 0 0 0))
   )
-  (wire (pts (xy 80.01 27.94) (xy 80.01 44.45))
+  (wire (pts (xy 82.55 27.94) (xy 82.55 44.45))
     (stroke (width 0) (type default) (color 0 0 0 0))
   )
@@
     )
   )
-  (global_label "CONTROL" (shape input) (at 71.12 52.07 180) (fields_autoplaced)
+  (global_label "CONTROL" (shape input) (at 67.31 52.07 180) (fields_autoplaced)
     (effects (font (size 1.27 1.27)) (justify right))
-    (property "Intersheet References" "${INTERSHEET_REFS}" (id 0) (at 60.1798 51.9906 0)
+    (property "Intersheet References" "${INTERSHEET_REFS}" (id 0) (at 56.3698 51.9906 0)
       (effects (font (size 1.27 1.27)) (justify right) hide)
     )
@@
     (pin "3")
   )
-  (symbol (lib_id "Device:R") (at 80.01 48.26 0) (unit 1)
-    (in_bom yes) (on_board yes) (fields_autoplaced)
-    (property "Reference" "R3" (id 0) (at 82.55 46.9899 0)
-      (effects (font (size 1.27 1.27)) (justify left))
-    )
-    (property "Value" "10k" (id 1) (at 82.55 49.5299 0)
-      (effects (font (size 1.27 1.27)) (justify left))
-    )
-    (property "Footprint" "" (id 2) (at 78.232 48.26 90)
-      (effects (font (size 1.27 1.27)) hide)
-    )
-    (property "Datasheet" "~" (id 3) (at 80.01 48.26 0)
+  (symbol (lib_id "Device:R") (at 82.55 48.26 0) (unit 1)
+    (in_bom yes) (on_board yes) (fields_autoplaced)
+    (property "Reference" "R3" (id 0) (at 85.09 46.9899 0)
+      (effects (font (size 1.27 1.27)) (justify left))
+    )
+    (property "Value" "10k" (id 1) (at 85.09 49.5299 0)
+      (effects (font (size 1.27 1.27)) (justify left))
+    )
+    (property "Footprint" "" (id 2) (at 80.772 48.26 90)
+      (effects (font (size 1.27 1.27)) hide)
+    )
+    (property "Datasheet" "~" (id 3) (at 82.55 48.26 0)
+      (effects (font (size 1.27 1.27)) hide)
+    )
+    (pin "1")
+    (pin "2")
+  )
+  (symbol (lib_id "Device:R") (at 74.93 52.07 90) (unit 1)
+    (in_bom yes) (on_board yes) (fields_autoplaced)
+    (property "Reference" "R9" (id 0) (at 74.93 45.72 90))
+    (property "Value" "100" (id 1) (at 74.93 48.26 90))
+    (property "Footprint" "" (id 2) (at 74.93 53.848 90)
+      (effects (font (size 1.27 1.27)) hide)
+    )
+    (property "Datasheet" "~" (id 3) (at 74.93 52.07 0)
       (effects (font (size 1.27 1.27)) hide)
     )
@@
       (reference "R8") (unit 1) (value "200") (footprint "")
     )
+    (path "/a16285e2-5718-43ab-89ab-6ed8d0e4e8ca"
+      (reference "R9") (unit 1) (value "100") (footprint "")
+    )
     (path "/10122f7b-475c-4599-a088-80ef527706a8"
